Commit message: intermediate (working) state from 1 month ago

File: ros2_description_solo/urdf/leg.xacro (robot description, xacro)
@@ -19,5 +19,5 @@
                 <parent link="base_link"/>
                 <child link="${prefix}_SHOULDER"/>
-                <limit effort="1000" lower="-3.14159" upper="3.14159" velocity="2"/>
+                <limit effort="1000" lower="-3.14159" upper="3.14159" velocity="80"/>
                 <!-- joints rotates around the x-axis -->
                 <axis xyz="1 0 0"/>
@@ -39,6 +39,5 @@
                     </xacro:if>
                 </xacro:unless>
-                <!-- pybullet simulation parameters -->
-                <dynamics damping="0.0" friction="0.0"/>
+                <dynamics damping="0.1" friction="0.0"/>
             </joint>
             <link name="${prefix}_SHOULDER">
@@ -85,5 +84,5 @@
                             <origin xyz="0.01950 0 0" rpy="0 0 0"/>
                             <geometry>
-                                <mesh filename="file://$(find ros2_description_solo)/meshes/${mesh_ext}/solo12/solo12_hip_fe_fl.${mesh_ext}"/>
+                                <mesh filename="file://$(find ros2_description_solo)/meshes/${mesh_ext}/solo12/solo12_hip_fe_fl-collision.${mesh_ext}"/>
                             </geometry>
                         </xacro:if>
@@ -91,5 +90,5 @@
                             <origin xyz="-0.01950 0 0" rpy="0 0 0"/>
                             <geometry>
-                                <mesh filename="file://$(find ros2_description_solo)/meshes/${mesh_ext}/solo12/solo12_hip_fe_hl.${mesh_ext}"/>
+                                <mesh filename="file://$(find ros2_description_solo)/meshes/${mesh_ext}/solo12/solo12_hip_fe_hl-collision.${mesh_ext}"/>
                             </geometry>
                         </xacro:unless>
@@ -99,5 +98,5 @@
                             <origin xyz="0.01950 0 0" rpy="0 0 0"/>
                             <geometry>
-                                <mesh filename="file://$(find ros2_description_solo)/meshes/${mesh_ext}/solo12/solo12_hip_fe_fr.${mesh_ext}"/>
+                                <mesh filename="file://$(find ros2_description_solo)/meshes/${mesh_ext}/solo12/solo12_hip_fe_fr-collision.${mesh_ext}"/>
                             </geometry>
                         </xacro:if>
@@ -105,5 +104,5 @@
                             <origin xyz="-0.01950 0 0" rpy="0 0 0"/>
                             <geometry>
-                                <mesh filename="file://$(find ros2_description_solo)/meshes/${mesh_ext}/solo12/solo12_hip_fe_hr.${mesh_ext}"/>
+                                <mesh filename="file://$(find ros2_description_solo)/meshes/${mesh_ext}/solo12/solo12_hip_fe_hr-collision.${mesh_ext}"/>
                             </geometry>
                         </xacro:unless>
@@ -152,5 +151,5 @@
                 <parent link="${prefix}_SHOULDER"/>
                 <child link="${prefix}_UPPER_LEG"/>
-                <limit effort="1000" lower="-3.14159" upper="3.14159" velocity="2"/>
+                <limit effort="1000" lower="-3.14159" upper="3.14159" velocity="80"/>
                 <!-- joints rotates around the y-axis -->
                 <axis xyz="0 1 0"/>
@@ -162,6 +161,5 @@
                     <origin xyz="0 ${HAA_2_HFE_y} 0" rpy="0 0 0"/>
                 </xacro:unless>
-                <!-- pybullet simulation parameters -->
-                <dynamics damping="0.0" friction="0.0"/>
+                <dynamics damping="0.1" friction="0.0"/>
             </joint>
         </xacro:if>
@@ -171,5 +169,5 @@
                 <parent link="base_link"/>
                 <child link="${prefix}_UPPER_LEG"/>
-                <limit effort="1000" lower="-3.14159" upper="3.14159" velocity="2"/>
+                <limit effort="1000" lower="-3.14159" upper="3.14159" velocity="80"/>
                 <!-- joints rotates around the y-axis -->
                 <axis xyz="0 1 0"/>
@@ -191,6 +189,5 @@
                     </xacro:if>
                 </xacro:unless>
-                <!-- pybullet simulation parameters -->
-<!--                <dynamics damping="0.0" friction="0.01"/>-->
+                <dynamics damping="0.1" friction="0.0"/>
             </joint>
         </xacro:unless>
@@ -237,8 +234,8 @@
                 <geometry>
                     <xacro:unless value="${is_right}">
-                        <mesh filename="file://$(find ros2_description_solo)/meshes/${mesh_ext}/with_foot/solo_upper_leg_left_side.${mesh_ext}"/>
-                    </xacro:unless>
-                    <xacro:if value="${is_right}">
-                        <mesh filename="file://$(find ros2_description_solo)/meshes/${mesh_ext}/with_foot/solo_upper_leg_right_side.${mesh_ext}"/>
+                        <mesh filename="file://$(find ros2_description_solo)/meshes/${mesh_ext}/with_foot/solo_upper_leg_left_side-collision.${mesh_ext}"/>
+                    </xacro:unless>
+                    <xacro:if value="${is_right}">
+                        <mesh filename="file://$(find ros2_description_solo)/meshes/${mesh_ext}/with_foot/solo_upper_leg_right_side-collision.${mesh_ext}"/>
                     </xacro:if>
                 </geometry>
@@ -257,5 +254,5 @@
             <parent link="${prefix}_UPPER_LEG"/>
             <child link="${prefix}_LOWER_LEG"/>
-            <limit effort="1000" lower="-3.14159" upper="3.14159" velocity="2"/>
+            <limit effort="1000" lower="-3.14159" upper="3.14159" velocity="80"/>
             <!-- joints rotates around the y-axis -->
             <axis xyz="0 1 0"/>
@@ -277,6 +274,5 @@
                 </xacro:if>
             </xacro:unless>
-            <!-- pybullet simulation parameters -->
-<!--            <dynamics damping="0.0" friction="0.0"/>-->
+            <dynamics damping="0.1" friction="0.0"/>
         </joint>
         <link name="${prefix}_LOWER_LEG">
@@ -322,8 +318,8 @@
                 <geometry>
                     <xacro:unless value="${is_right}">
-                        <mesh filename="file://$(find ros2_description_solo)/meshes/${mesh_ext}/with_foot/solo_lower_leg_left_side.${mesh_ext}"/>
-                    </xacro:unless>
-                    <xacro:if value="${is_right}">
-                        <mesh filename="file://$(find ros2_description_solo)/meshes/${mesh_ext}/with_foot/solo_lower_leg_right_side.${mesh_ext}"/>
+                        <mesh filename="file://$(find ros2_description_solo)/meshes/${mesh_ext}/with_foot/solo_lower_leg_left_side-collision.${mesh_ext}"/>
+                    </xacro:unless>
+                    <xacro:if value="${is_right}">
+                        <mesh filename="file://$(find ros2_description_solo)/meshes/${mesh_ext}/with_foot/solo_lower_leg_right_side-collision.${mesh_ext}"/>
                     </xacro:if>
                 </geometry>
@@ -351,7 +347,6 @@
             </xacro:if>
             <!-- Limits (usefull?) -->
-            <limit effort="1000" lower="-3.14159" upper="3.14159" velocity="2"/>
-            <!-- pybullet simulation parameters -->
-<!--            <dynamics damping="0.0" friction="0.0"/>-->
+            <limit effort="1000" lower="-3.14159" upper="3.14159" velocity="80"/>
+            <dynamics damping="0.1" friction="0.0"/>
         </joint>
         <link name="${prefix}_FOOT">
@@ -379,9 +374,10 @@
                 <origin xyz="0 0 0" rpy="0 0 0"/>
                 <geometry>
-                    <mesh filename="file://$(find ros2_description_solo)/meshes/${mesh_ext}/with_foot/solo_foot.${mesh_ext}"/>
-                </geometry>
-                <material name="${color_name}">
-                    <color rgba="${color} ${opacity}"/>
-                </material>
+                    <mesh filename="file://$(find ros2_description_solo)/meshes/${mesh_ext}/with_foot/solo_foot-collision.${mesh_ext}"/>
+                </geometry>
+                <material name="${color_name}">
+                    <color rgba="${color} ${opacity}"/>
+                </material>
+                <!--
                 <gazebo>
                     <surface>
@@ -408,4 +404,5 @@
                     </surface>
                 </gazebo>
+                -->
             </collision>
         </link> <!-- END LOWER LEG LINK -->
@@ -427,7 +424,13 @@
         </gazebo>
         <gazebo reference="${prefix}_FOOT">
-            <material>Gazebo/White</material>
 <!--            <selfCollide>true</selfCollide>-->
 <!--            <gravity>true</gravity>-->
+            <kp>1000000.0</kp>
+            <kd>1.0</kd>
+            <mu1>0.8</mu1>
+            <mu2>0.8</mu2>
+            <maxVel>1.0</maxVel>
+            <minDepth>0.001</minDepth>
+            <material>Gazebo/FlatBlack</material>
         </gazebo>
     </xacro:macro>

File: ros2_description_solo/urdf/solo12.urdf.xacro (robot description, xacro)
@@ -1,9 +1,10 @@
 <?xml version="1.0" ?>
-<robot name="solo" xmlns:xacro="http://www.ros.org/wiki/xacro">
+<robot name="solo12" xmlns:xacro="http://www.ros.org/wiki/xacro">
     <xacro:property name="color_name" value="grey"/>
     <xacro:property name="color" value="0.8 0.8 0.8"/>
     <xacro:property name="opacity" value="1.0"/>
     <xacro:property name="mesh_ext" value="stl"/>
-    <xacro:arg name="use_fake_hardware" default="true"/>
+    <xacro:arg name="use_fake_hardware" default="false"/>
+    <xacro:arg name="use_sim" default="false"/>
     <xacro:arg name="prefix" default=""/>
     <!-- remove if using crane -->
@@ -50,5 +51,5 @@
             <origin xyz="0 0 0" rpy="0 0 0"/>
             <geometry>
-                <mesh filename="file://$(find ros2_description_solo)/meshes/${mesh_ext}/solo12/solo_12_base.${mesh_ext}"/>
+                <mesh filename="file://$(find ros2_description_solo)/meshes/${mesh_ext}/solo12/solo_12_base-collision.${mesh_ext}"/>
             </geometry>
             <material name="${color_name}">
@@ -106,10 +107,8 @@
     <gazebo reference="base_link">
         <material>Gazebo/White</material>
-<!--        <selfCollide>true</selfCollide>-->
-        <!--        <gravity>true</gravity>-->
     </gazebo>
     <gazebo>
         <plugin filename="libgazebo_ros2_control.so" name="gazebo_ros2_control">
-            <parameters>$(find ros2_control_solo_bringup)/config/solo_gazebo_forward_controller_position.yaml
+            <parameters>$(find ros2_control_solo_bringup)/config/solo_gazebo_test_controllers_mod.yaml
             </parameters>
         </plugin>
